File: hw/RC_module.sch (EAGLE design)
At the start: 44 parts, among them J1 GROVE-4P-2.0-3470130P1, J2 GROVE-4P-2.0-3470130P1, X1 22-23-2021

Commit message: added R values
Parts:
- R2: value 10k -> 330
- RN1: value (none) -> 330
Changed lines of the file:
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@@
 <part name="P+13" library="supply" deviceset="+V" device=""/>
 <part name="P+14" library="supply" deviceset="+V" device=""/>
-<part name="RN1" library="dp_devices" deviceset="RESISTOR_ARRAY_4" device=""/>
+<part name="RN1" library="dp_devices" deviceset="RESISTOR_ARRAY_4" device="" value="330"/>
 <part name="RN2" library="dp_devices" deviceset="RESISTOR_ARRAY_4" device=""/>
 <part name="RN3" library="dp_devices" deviceset="RESISTOR_ARRAY_4" device=""/>
@@
 <part name="P+4" library="supply" deviceset="+V" device=""/>
 <part name="P+5" library="supply" deviceset="+V" device=""/>
-<part name="R2" library="rcl" deviceset="R-EU_" device="R0603" value="10k"/>
+<part name="R2" library="rcl" deviceset="R-EU_" device="R0603" value="330"/>
 <part name="R4" library="rcl" deviceset="R-EU_" device="R0603" value="10k"/>
 <part name="R5" library="rcl" deviceset="R-EU_" device="R0603" value="10k"/>

Commit message: small fixes
Parts:
- removed R4, R5: 10k, rcl:R-EU_R0603
- removed ZD1: (no value), dp_devices:ZENERSOD-323F
- added C10: (no value), rcl:CPOL-EUB/3528-21R
Connections:
- net +V: now also C10.+; no longer R4.2
- net GND: now also C10.-; no longer R5.1, ZD1.A
- net VSENSE: no longer R4.1, R5.2, ZD1.C
Other:
- moved on the sheet: X1-2
Changed lines of the file:
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@@
 <?xml version="1.0" encoding="utf-8"?>
 <!DOCTYPE eagle SYSTEM "eagle.dtd">
-<eagle version="6.4">
+<eagle version="7.2.0">
 <drawing>
 <settings>
@@
 <part name="P+5" library="supply" deviceset="+V" device=""/>
 <part name="R2" library="rcl" deviceset="R-EU_" device="R0603" value="330"/>
-<part name="R4" library="rcl" deviceset="R-EU_" device="R0603" value="10k"/>
-<part name="R5" library="rcl" deviceset="R-EU_" device="R0603" value="10k"/>
-<part name="ZD1" library="dp_devices" deviceset="ZENER" device="SOD-323F"/>
-<part name="GND28" library="supply1" deviceset="GND" device=""/>
-<part name="GND32" library="supply1" deviceset="GND" device=""/>
-<part name="P+15" library="supply" deviceset="+V" device=""/>
+<part name="C10" library="rcl" deviceset="CPOL-EU" device="B/3528-21R"/>
 </parts>
 <sheets>
@@
 <instance part="RN3" gate="A" x="327.66" y="154.94"/>
 <instance part="X1" gate="-1" x="208.28" y="86.36"/>
-<instance part="X1" gate="-2" x="208.28" y="81.28"/>
+<instance part="X1" gate="-2" x="208.28" y="78.74"/>
 <instance part="JP9" gate="G$1" x="210.82" y="152.4" rot="MR180"/>
 <instance part="GND33" gate="1" x="203.2" y="144.78"/>
 <instance part="P+1" gate="1" x="203.2" y="162.56"/>
-<instance part="GND35" gate="1" x="203.2" y="76.2"/>
+<instance part="GND35" gate="1" x="203.2" y="73.66"/>
 <instance part="P+2" gate="1" x="203.2" y="91.44"/>
 <instance part="JP7" gate="G$1" x="299.72" y="182.88" rot="MR180"/>
@@
 <instance part="P+5" gate="1" x="335.28" y="193.04"/>
 <instance part="R2" gate="G$1" x="195.58" y="124.46" rot="R180"/>
-<instance part="R4" gate="G$1" x="436.88" y="226.06" rot="R180"/>
-<instance part="R5" gate="G$1" x="444.5" y="220.98" rot="R90"/>
-<instance part="ZD1" gate="G$1" x="454.66" y="220.98" rot="R90"/>
-<instance part="GND28" gate="1" x="444.5" y="213.36"/>
-<instance part="GND32" gate="1" x="454.66" y="213.36"/>
-<instance part="P+15" gate="1" x="429.26" y="231.14"/>
+<instance part="C10" gate="G$1" x="203.2" y="83.82"/>
 </instances>
 <busses>
@@
 <segment>
 <pinref part="GND35" gate="1" pin="GND"/>
-<wire x1="203.2" y1="81.28" x2="203.2" y2="78.74" width="0.1524" layer="91"/>
+<wire x1="203.2" y1="78.74" x2="203.2" y2="76.2" width="0.1524" layer="91"/>
 <pinref part="X1" gate="-2" pin="S"/>
-<wire x1="203.2" y1="81.28" x2="205.74" y2="81.28" width="0.1524" layer="91"/>
+<wire x1="203.2" y1="78.74" x2="205.74" y2="78.74" width="0.1524" layer="91"/>
+<pinref part="C10" gate="G$1" pin="-"/>
+<junction x="203.2" y="78.74"/>
 </segment>
 <segment>
@@
 <wire x1="294.64" y1="180.34" x2="292.1" y2="180.34" width="0.1524" layer="91"/>
 <wire x1="292.1" y1="180.34" x2="292.1" y2="177.8" width="0.1524" layer="91"/>
-</segment>
-<segment>
-<pinref part="R5" gate="G$1" pin="1"/>
-<pinref part="GND28" gate="1" pin="GND"/>
-</segment>
-<segment>
-<pinref part="ZD1" gate="G$1" pin="A"/>
-<pinref part="GND32" gate="1" pin="GND"/>
-<wire x1="454.66" y1="215.9" x2="454.66" y2="218.44" width="0.1524" layer="91"/>
 </segment>
 </net>
@@
 <pinref part="X1" gate="-1" pin="S"/>
 <wire x1="203.2" y1="86.36" x2="205.74" y2="86.36" width="0.1524" layer="91"/>
+<pinref part="C10" gate="G$1" pin="+"/>
+<junction x="203.2" y="86.36"/>
 </segment>
 <segment>
@@
 <wire x1="335.28" y1="182.88" x2="335.28" y2="190.5" width="0.1524" layer="91"/>
 </segment>
-<segment>
-<pinref part="R4" gate="G$1" pin="2"/>
-<wire x1="431.8" y1="226.06" x2="429.26" y2="226.06" width="0.1524" layer="91"/>
-<pinref part="P+15" gate="1" pin="+V"/>
-<wire x1="429.26" y1="226.06" x2="429.26" y2="228.6" width="0.1524" layer="91"/>
-</segment>
 </net>
 <net name="N$11" class="0">
@@
 <label x="40.64" y="175.26" size="1.778" layer="95" rot="MR270"/>
 </segment>
-<segment>
-<pinref part="R4" gate="G$1" pin="1"/>
-<pinref part="R5" gate="G$1" pin="2"/>
-<wire x1="444.5" y1="226.06" x2="441.96" y2="226.06" width="0.1524" layer="91"/>
-<wire x1="444.5" y1="226.06" x2="454.66" y2="226.06" width="0.1524" layer="91"/>
-<junction x="444.5" y="226.06"/>
-<pinref part="ZD1" gate="G$1" pin="C"/>
-<wire x1="454.66" y1="226.06" x2="459.74" y2="226.06" width="0.1524" layer="91"/>
-<wire x1="454.66" y1="223.52" x2="454.66" y2="226.06" width="0.1524" layer="91"/>
-<junction x="454.66" y="226.06"/>
-<label x="459.74" y="226.06" size="1.778" layer="95"/>
-</segment>
-</net>
+</net>
