File: hw/RC_module.sch (EAGLE design)
At the start: 42 parts, among them J1 GROVE-4P-2.0-3470130P1, J2 GROVE-4P-2.0-3470130P1, X1 22-23-2021

Commit message: Added logo to bottom silkscreen
Connections:
- net GND: now also LED1.C; no longer LED1.A
- net N$4: now also LED1.A; no longer LED1.C
Other:
- moved on the sheet: LED1
Changed lines of the file:
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@@
 <instance part="C7" gate="G$1" x="124.46" y="71.12"/>
 <instance part="GND22" gate="1" x="124.46" y="63.5"/>
-<instance part="LED1" gate="G$1" x="22.86" y="114.3" rot="R180"/>
+<instance part="LED1" gate="G$1" x="22.86" y="116.84"/>
 <instance part="R1" gate="G$1" x="22.86" y="127" rot="R90"/>
 <instance part="GND16" gate="1" x="81.28" y="10.16"/>
@@
 </segment>
 <segment>
-<pinref part="LED1" gate="G$1" pin="A"/>
-<pinref part="GND13" gate="1" pin="GND"/>
-</segment>
-<segment>
 <wire x1="78.74" y1="66.04" x2="76.2" y2="66.04" width="0.1524" layer="91"/>
 <pinref part="GND10" gate="1" pin="GND"/>
@@
 <wire x1="294.64" y1="180.34" x2="292.1" y2="180.34" width="0.1524" layer="91"/>
 <wire x1="292.1" y1="180.34" x2="292.1" y2="177.8" width="0.1524" layer="91"/>
+</segment>
+<segment>
+<pinref part="GND13" gate="1" pin="GND"/>
+<pinref part="LED1" gate="G$1" pin="C"/>
 </segment>
 </net>
@@
 <segment>
 <pinref part="R1" gate="G$1" pin="1"/>
-<pinref part="LED1" gate="G$1" pin="C"/>
 <wire x1="22.86" y1="119.38" x2="22.86" y2="121.92" width="0.1524" layer="91"/>
-</segment>
-</net>
+<pinref part="LED1" gate="G$1" pin="A"/>
+</segment>
+</net>
